File: AlienWhoopF7-ESP32.sch (EAGLE design)
At the start: 62 parts, among them IC1 ESP32-WROOM-32E-N4, M1 53047-0210, M2 53047-0210, M3 53047-0210, M4 53047-0210, Q1 IRLML6402, Q2 FDMA410NZT, Q3 FDMA410NZT, Q4 FDMA410NZT, Q5 FDMA410NZT, Q6 MMBT3904, Q7 MMBT3904, U1 TPS63001, U2 MPU-6500, U3 MX25L6406EM2I-12G, U5 CH340C

Commit message: Switch to ESP32-MINI-1 and add generated placement-study board
The layout pass falsified the WROOM-32E: the motor-plug through-holes
leave a 14.4mm corridor and the module is 18mm wide. The ESP32-MINI-1
(13.2mm, same ESP32-U4WDH silicon family, same esp32 IDF target, 4MB
in-package flash) fits with the antenna fully off the board edge. Its
in-package flash consumes GPIO16/17, so the receiver UART moves to
IO9/IO10 (the native U1RXD/U1TXD).

AlienWhoopF7-ESP32.brd is a generated transplant of the original
layout: all surviving parts keep their positions, GND/3V3 pours and
unmoved power copper carry over, the gyro moves to board center on
the bottom, the CH340C cluster takes the deleted inverter space.
Verified collision-free at 0.2mm with through-hole punch-through and
module-body keepout checked; 34 module-bound nets are airwires for an
interactive routing pass in Eagle.

Co-Authored-By: Claude Fable 5 <noreply@anthropic.com>
Parts:
- IC1: value ESP32-WROOM-32E-N4 -> ESP32-MINI-1-N4; device esp32:ESP32-WROOM-32E -> esp32:ESP32-MINI-1
Connections:
- net IO36: now also IC1.IO36; no longer IC1.SENSOR_VP
- net UART2_RX: now also IC1.IO9; no longer IC1.IO16
- net UART2_TX: now also IC1.IO10; no longer IC1.IO17
Other:
- note added: "MCU: ESP32-MINI-1 (13.2mm wide - the WROOM-32E does not fit between the motor plug through-holes). Deleted: Y1 resonator, U4 SBUS inverter (UART inverts in silicon), C7/C10/C15 dual-MCU selection sites."
- note added: "Motors: M1=IO25 M2=IO27 M3=IO33 M4=IO32. Pads: RX2/TX2=IO9/IO10 (SBUS; IO16/IO17 do not exist on this module), RX3/TX3=IO21/IO22 (UART1/console), IO4=RMT, IO36=spare ADC."
- note removed: "MCU: ESP32-WROOM-32E replaces STM32F405/F722 (LQFP64). Deleted: Y1 resonator, U4 SBUS inverter (UART inverts in silicon), C7/C10/C15 VCAP caps."
- note removed: "Motors: M1=IO25 M2=IO27 M3=IO33 M4=IO32. Pads: RX2/TX2=IO16/IO17 (UART2, SBUS), RX3/TX3=IO21/IO22 (UART1/console), IO4=RMT, IO36=spare ADC."
- moved on the sheet: C1, C11, C12, C13, C14, C16, C17, C18, C19, C2, C3, C4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
